Commit message: add camera support

File: mara_description/urdf/camera_gripper.urdf.xacro (robot description, xacro)
@@ -12,5 +12,5 @@
         <origin rpy="0 0 0" xyz="0 0 0"/>
         <geometry>
-          <mesh filename="package://mara_description/meshes/ROBOTIQ_Gripper_Adapter.dae" scale="0.1 0.1 0.1"/>
+          <mesh filename="package://mara_description/meshes/ROBOTIQ_Gripper_Adapter.dae" scale="0.001 0.001 0.001"/>
         </geometry>
         <material name="Gazebo/Wood">
@@ -21,5 +21,5 @@
         <origin rpy="0 0 0" xyz="0 0 0"/>
         <geometry>
-          <mesh filename="package://mara_description/meshes/ROBOTIQ_Gripper_Adapter.dae" scale="0.1 0.1 0.1"/>
+          <mesh filename="package://mara_description/meshes/ROBOTIQ_Gripper_Adapter.dae" scale="0.001 0.001 0.001"/>
         </geometry>
       </collision>
@@ -38,5 +38,5 @@
         <origin rpy="0 0 0" xyz="0 0 0"/>
         <geometry>
-          <mesh filename="package://mara_description/meshes/Camera_Support_1.dae" scale="0.1 0.1 0.1"/>
+          <mesh filename="package://mara_description/meshes/Camera_Support_1.dae" scale="0.001 0.001 0.001"/>
         </geometry>
         <material name="Gazebo/Wood">
@@ -47,5 +47,5 @@
         <origin rpy="0 0 0" xyz="0 0 0"/>
         <geometry>
-          <mesh filename="package://mara_description/meshes/Camera_Support_1.dae" scale="0.1 0.1 0.1"/>
+          <mesh filename="package://mara_description/meshes/Camera_Support_1.dae" scale="0.001 0.001 0.001"/>
         </geometry>
       </collision>
@@ -64,5 +64,5 @@
         <origin rpy="0 0 0" xyz="0 0 0"/>
         <geometry>
-          <mesh filename="package://mara_description/meshes/Camera_Support_2.dae" scale="0.1 0.1 0.1"/>
+          <mesh filename="package://mara_description/meshes/Camera_Support_2.dae" scale="0.001 0.001 0.001"/>
         </geometry>
         <material name="Gazebo/Wood">
@@ -73,5 +73,5 @@
         <origin rpy="0 0 0" xyz="0 0 0"/>
         <geometry>
-          <mesh filename="package://mara_description/meshes/Camera_Support_2.dae" scale="0.1 0.1 0.1"/>
+          <mesh filename="package://mara_description/meshes/Camera_Support_2.dae" scale="0.001 0.001 0.001"/>
         </geometry>
       </collision>
@@ -91,5 +91,5 @@
       <child link="${prefix}mara_camera_support2_link"/>
     </joint>
-    <!-- <xacro:sensor_d435 prefix="${prefix}mara_camera_support2_link" origin="mcs2l"/> -->
+    <!-- <xacro:sensor_d435 prefix="${prefix}mara_camera_support2_link"/> -->
   </xacro:macro>
 </robot>

File: mara_description/urdf/d435.urdf.xacro (robot description, xacro)
@@ -7,5 +7,5 @@
 -->
 <robot name="sensor_d435" xmlns:xacro="http://ros.org/wiki/xacro">
-  <xacro:macro name="sensor_d435" params="parent *origin">
+  <xacro:macro name="sensor_d435" params="parent">
     <xacro:property name="M_PI" value="3.1415926535897931" />
     <!-- The following values are approximate, and the camera node
