Commit message: fix xacro files

File: mara_description/urdf/mara_gazebo.urdf.xacro (robot description, xacro)
@@ -3,34 +3,12 @@
   <xacro:macro name="mara_gazebo" params="prefix">
     <gazebo>
-      <plugin name="mara_joint_state" filename="libgazebo_ros_joint_state_publisher.so">
-    		<ros>
-    			<argument>~/out:=joint_states</argument>
-    		</ros>
-    		<update_rate>25</update_rate>
-    		<joint_name>motor1</joint_name>
-    		<joint_name>motor2</joint_name>
-    		<joint_name>motor3</joint_name>
-    		<joint_name>motor4</joint_name>
-    		<joint_name>motor5</joint_name>
-        <joint_name>motor6</joint_name>
-        <joint_name>joint_finger</joint_name>
-    	</plugin>
-      <plugin name="hros_actuation_servomotor_000000000001" filename="libmara_gazebo_joint_training_plugin.so">
+      <plugin name="hros_actuation_servomotor_00000000000" filename="libmara_gazebo_joint_training_plugin.so">
         <ros></ros>
         <axis1>motor2</axis1>
         <axis2>motor1</axis2>
-        <type>series14</type>
-      </plugin>
-      <plugin name="hros_actuation_servomotor_000000000002" filename="libmara_gazebo_joint_training_plugin.so">
-        <ros></ros>
-        <axis1>motor3</axis1>
-        <axis2>motor4</axis2>
-        <type>series17</type>
-      </plugin>
-      <plugin name="hros_actuation_servomotor_000000000003" filename="libmara_gazebo_joint_training_plugin.so">
-        <ros></ros>
-        <axis1>motor5</axis1>
-        <axis2>motor6</axis2>
-        <type>series20</type>
+        <axis3>motor3</axis3>
+        <axis4>motor4</axis4>
+        <axis5>motor5</axis5>
+        <axis6>motor6</axis6>
       </plugin>
     </gazebo>

File: mara_description/urdf/mara_robot_gripper_140.urdf (robot description, URDF)
Before this commit: robot mara, 24 links, 23 joints
Links:
- added link robotiq_adapter_link, mass 0.22652; collision mesh filename=package://robotiq_140_gripper_description/meshes/hros_robot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 scale=0.001 0.001 0.001; visual mesh filename=package://robotiq_140_gripper_description/meshes/hros_robot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 scale=0.001 0.001 0.001
Joints:
- added joint base_adapter_to_base_robotiq_joint: type fixed, parent robotiq_adapter_link, child robotiq_arg2f_base_link, origin xyz= 0 0 0.03653 rpy=0 0 0
- joint end_effector_adapter_to_robotiq: child robotiq_arg2f_base_link -> robotiq_adapter_link

File: mara_description/urdf/mara_robot_gripper_140.urdf.xacro (robot description, xacro)
@@ -19,5 +19,5 @@
     <origin rpy="0 0 1.57" xyz=" 0 0 0.03653"/>
     <parent link="motor6_link"/>
-    <child link="robotiq_arg2f_base_link"/>
+    <child link="robotiq_adapter_link"/>
   </joint>
   <joint name="world_to_table_joint" type="fixed">
