Commit message: add camera urdf

File: mara_description/urdf/camera_gripper_support.urdf.xacro (robot description, xacro)
@@ -1,6 +1,5 @@
 <?xml version="1.0"?>
 <robot xmlns:xacro="http://ros.org/wiki/xacro">
-  <xacro:include filename="$(find mara_description)/urdf/d435.urdf.xacro" />
-  <xacro:macro name="mara_camera_gripper" params="prefix">
+  <xacro:macro name="mara_camera_gripper_support" params="prefix">
     <link name="${prefix}mara_gripper_adapter">
       <inertial>
@@ -26,5 +25,5 @@
     </link>
     <gazebo reference="${prefix}mara_gripper_adapter">
-      <material>Gazebo/Grey</material>
+      <material>Gazebo/Black</material>
       <selfCollide>True</selfCollide>
     </gazebo>
@@ -52,5 +51,5 @@
     </link>
     <gazebo reference="${prefix}mara_camera_support1_link">
-      <material>Gazebo/Grey</material>
+      <material>Gazebo/Black</material>
       <selfCollide>True</selfCollide>
     </gazebo>
@@ -78,5 +77,5 @@
     </link>
     <gazebo reference="${prefix}mara_camera_support2_link">
-      <material>Gazebo/Grey</material>
+      <material>Gazebo/Black</material>
       <selfCollide>True</selfCollide>
     </gazebo>
@@ -91,5 +90,4 @@
       <child link="${prefix}mara_camera_support2_link"/>
     </joint>
-    <!-- <xacro:sensor_d435/> -->
   </xacro:macro>
 </robot>

File: mara_description/urdf/mara_robot_gripper_140_camera.urdf (robot description, URDF)
Before this commit: robot mara, 27 links, 26 joints
Links:
- added link camera_color
- added link camera_ir_projector
- added link camera_left_depth
- added link camera_link, mass 0.564; collision mesh filename=package://mara_description/meshes/Intel_RealSense_Depth_Cam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 scale=0.001 0.001 0.001; visual mesh filename=package://mara_description/meshes/Intel_RealSense_Depth_Cam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 scale=0.001 0.001 0.001
- added link camera_right_depth
- added link robotiq_adapter_link, mass 0.22652; collision mesh filename=package://robotiq_140_gripper_description/meshes/hros_robot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 scale=0.001 0.001 0.001; visual mesh filename=package://robotiq_140_gripper_description/meshes/hros_robot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 scale=0.001 0.001 0.001
- link ee_link: geometry 
Joints:
- added joint base_adapter_to_base_robotiq_joint: type fixed, parent robotiq_adapter_link, child robotiq_arg2f_base_link, origin xyz= 0 0 0.03653 rpy=0 0 0
- added joint camera_support2_to_camera_link: type fixed, parent mara_camera_support2_link, child camera_link, origin xyz=0 0.018 0.012 rpy=0 0 0
- added joint camera_to_color: type fixed, parent camera_link, child camera_color, origin xyz=-0.0325 0.0214 0.0 rpy=0.0 0.0 1.57
- added joint camera_to_ir_projector: type fixed, parent camera_link, child camera_ir_projector, origin xyz=0.0115 0.0214 0.0 rpy=0 0 0
- added joint camera_to_left_depth: type fixed, parent camera_link, child camera_left_depth, origin xyz=-0.0175 0.024 0.0 rpy=0 0 0
- added joint camera_to_right_depth: type fixed, parent camera_link, child camera_right_depth, origin xyz=0.0325 0.024 0.0 rpy=1.57 0 0
- joint ee_link: origin xyz=0 0.0 0.24 rpy=0 0 0 -> xyz=0 0.0 0.24 rpy=0 -1.57 0
- joint end_effector_adapter_to_robotiq: child robotiq_arg2f_base_link -> robotiq_adapter_link; origin xyz= 0 0 0.03653 rpy=0 0 1.57 -> xyz= 0 0 0 rpy=0 0 1.57
- joint motor6_link-tool0_fixed_joint: origin xyz=0 0.0 0.24 rpy=0 0 0 -> xyz=0 0.0 0.24 rpy=0 -1.57 0

File: mara_description/urdf/mara_robot_gripper_140_camera.urdf.xacro (robot description, xacro)
@@ -6,5 +6,6 @@
   <!-- mara -->
   <xacro:include filename="$(find mara_description)/urdf/mara.urdf.xacro" />
-  <xacro:include filename="$(find mara_description)/urdf/camera_gripper.urdf.xacro" />
+  <xacro:include filename="$(find mara_description)/urdf/camera_gripper_support.urdf.xacro" />
+  <xacro:include filename="$(find mara_description)/urdf/rs_d435.urdf.xacro" />
   <!-- robotiq 140 gripper -->
   <xacro:include filename="$(find robotiq_140_gripper_description)/urdf/robotiq_140.urdf.xacro" />
@@ -12,5 +13,6 @@
   <!-- arm -->
   <xacro:mara_robot prefix="" ee_link_distance="0.24"/>
-  <xacro:mara_camera_gripper prefix="" />
+  <xacro:mara_camera_gripper_support prefix="" />
+  <xacro:rs_d435_camera prefix="" />
   <xacro:robotiq_gripper prefix="mara" />
   <xacro:table prefix="" />
@@ -22,7 +24,12 @@
   </joint>
   <joint name="end_effector_adapter_to_robotiq" type="fixed">
-    <origin rpy="0 0 1.57" xyz=" 0 0 0.03653"/>
+    <origin rpy="0 0 1.57" xyz=" 0 0 0"/>
     <parent link="mara_gripper_adapter"/>
-    <child link="robotiq_arg2f_base_link"/>
+    <child link="robotiq_adapter_link"/>
+  </joint>
+  <joint name="camera_support2_to_camera_link" type="fixed">
+    <origin rpy="0 0 0" xyz="0 0.018 0.012"/>
+    <parent link="mara_camera_support2_link"/>
+    <child link="camera_link"/>
   </joint>
   <joint name="world_to_table_joint" type="fixed">

Commit message: fix mass and inertia values

File: mara_description/urdf/camera_gripper_support.urdf.xacro (robot description, xacro)
@@ -5,6 +5,6 @@
       <inertial>
         <origin rpy="0 0 0" xyz="8.625E-08 -4.6583E-06 0.03145"/>
-        <mass value="7.033"/>
-        <inertia ixx="0.1478344" ixy="-0.00001" ixz="0.0" iyy="0.14782335" iyz="0.0" izz="0.29471799"/>
+        <mass value="0.1"/>
+        <inertia ixx="0.00739172" ixy="-0.00001" ixz="0.0" iyy="0.00739172" iyz="0.0" izz="0.0147358995"/>
       </inertial>
       <visual>
@@ -31,6 +31,6 @@
       <inertial>
         <origin rpy="0 0 0" xyz="8.625E-08 -4.6583E-06 0.03145"/>
-        <mass value="7.033"/>
-        <inertia ixx="0.1478344" ixy="-0.00001" ixz="0.0" iyy="0.14782335" iyz="0.0" izz="0.29471799"/>
+        <mass value="0.1"/>
+        <inertia ixx="0.00739172" ixy="-0.00001" ixz="0.0" iyy="0.00739172" iyz="0.0" izz="0.0147358995"/>
       </inertial>
       <visual>
@@ -57,6 +57,6 @@
       <inertial>
         <origin rpy="0 0 0" xyz="8.625E-08 -4.6583E-06 0.03145"/>
-        <mass value="7.033"/>
-        <inertia ixx="0.1478344" ixy="-0.00001" ixz="0.0" iyy="0.14782335" iyz="0.0" izz="0.29471799"/>
+        <mass value="0.1"/>
+        <inertia ixx="0.00739172" ixy="-0.00001" ixz="0.0" iyy="0.00739172" iyz="0.0" izz="0.0147358995"/>
       </inertial>
       <visual>

File: mara_description/urdf/mara_robot_gripper_140_camera.urdf (robot description, URDF)
Before this commit: robot mara, 33 links, 32 joints
Links:
- link mara_camera_support1_link: mass 7.033 -> 0.1
- link mara_camera_support2_link: mass 7.033 -> 0.1
- link mara_gripper_adapter: mass 7.033 -> 0.1
