Commit message: update run urdf

File: mara_description/urdf/mara_robot_gripper_140_run.urdf (robot description, URDF)
Before this commit: robot mara, 24 links, 23 joints
Links:
- added link robotiq_adapter_link, mass 0.22652; collision mesh filename=package://robotiq_140_gripper_description/meshes/hros_robot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 scale=0.001 0.001 0.001; visual mesh filename=package://robotiq_140_gripper_description/meshes/hros_robot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 scale=0.001 0.001 0.001
- link ee_link: geometry 
Joints:
- added joint base_adapter_to_base_robotiq_joint: type fixed, parent robotiq_adapter_link, child robotiq_arg2f_base_link, origin xyz= 0 0 0.03653 rpy=0 0 0
- joint ee_link: origin xyz=0 0.0 0.24 rpy=0 0 0 -> xyz=0 0.0 0.24 rpy=0 -1.57 0
- joint end_effector_adapter_to_robotiq: child robotiq_arg2f_base_link -> robotiq_adapter_link; origin xyz= 0 0 0.03653 rpy=0 0 1.57 -> xyz= 0 0 0 rpy=0 0 1.57
- joint motor6_link-tool0_fixed_joint: origin xyz=0 0.0 0.24 rpy=0 0 0 -> xyz=0 0.0 0.24 rpy=0 -1.57 0
