Commit message: fix mara_robot_gripper_140

File: mara_description/urdf/mara.urdf.xacro (robot description, xacro)
@@ -294,12 +294,4 @@
     </gazebo>
     <link name="${prefix}ee_link">
-      <visual>
-        <geometry>
-          <sphere radius="0.01"/>
-        </geometry>
-        <material name="Gazebo/Grey">
-          <color rgba="0. 0. 0. 1"/>
-        </material>
-      </visual>
     </link>
     <gazebo reference="${prefix}ee_link">
@@ -376,5 +368,5 @@
     </joint>
     <joint name="${prefix}ee_link" type="fixed">
-      <origin rpy="0 0 0" xyz="0 0.0 ${ee_link_distance}"/> <!-- 0.24 -->
+      <origin rpy="0 -1.57 0" xyz="0 0.0 ${ee_link_distance}"/> <!-- 0.24 -->
       <parent link="${prefix}motor6_link"/>
       <child link="${prefix}ee_link"/>
@@ -382,5 +374,5 @@
     <link name="${prefix}tool0"/>
     <joint name="${prefix}${prefix}motor6_link-tool0_fixed_joint" type="fixed">
-      <origin rpy="0 0 0" xyz="0 0.0 ${ee_link_distance}"/>
+      <origin rpy="0 -1.57 0" xyz="0 0.0 ${ee_link_distance}"/>
       <parent link="${prefix}${prefix}motor6_link"/>
       <child link="${prefix}tool0"/>

File: mara_description/urdf/mara_robot_gripper_140.urdf (robot description, URDF)
Before this commit: robot mara, 25 links, 24 joints
Links:
- link ee_link: geometry 
Joints:
- joint ee_link: origin xyz=0 0.0 0.24 rpy=0 0 0 -> xyz=0 0.0 0.24 rpy=0 -1.57 0
- joint end_effector_adapter_to_robotiq: origin xyz= 0 0 0.03653 rpy=0 0 1.57 -> xyz= 0 0 0 rpy=0 0 1.57
- joint motor6_link-tool0_fixed_joint: origin xyz=0 0.0 0.24 rpy=0 0 0 -> xyz=0 0.0 0.24 rpy=0 -1.57 0

File: mara_description/urdf/mara_robot_gripper_140.urdf.xacro (robot description, xacro)
@@ -17,5 +17,5 @@
   <link name="world" />
   <joint name="end_effector_adapter_to_robotiq" type="fixed">
-    <origin rpy="0 0 1.57" xyz=" 0 0 0.03653"/>
+    <origin rpy="0 0 1.57" xyz=" 0 0 0"/>
     <parent link="motor6_link"/>
     <child link="robotiq_adapter_link"/>

Commit message: add blue dot

File: mara_description/urdf/mara.urdf.xacro (robot description, xacro)
@@ -294,4 +294,12 @@
     </gazebo>
     <link name="${prefix}ee_link">
+      <visual>
+        <geometry>
+          <sphere radius="0.01"/>
+        </geometry>
+        <material name="Gazebo/Grey">
+          <color rgba="0. 0. 0. 1"/>
+        </material>
+      </visual>
     </link>
     <gazebo reference="${prefix}ee_link">

File: mara_description/urdf/mara_robot_gripper_140.urdf (robot description, URDF)
Before this commit: robot mara, 25 links, 24 joints
Links:
- link ee_link: geometry visual sphere radius=0.01

File: mara_description/urdf/mara_robot_gripper_140_run.urdf (robot description, URDF)
Before this commit: robot mara, 25 links, 24 joints
Links:
- link ee_link: geometry visual sphere radius=0.01
